Commit message: feat: Robotiq 2F-85 body visuals + slimmer sliding fingers, retune pick/place height
- gripper body/adapter use Robotiq 2F-85 meshes (MIT, from darshmenon/UR3_ROS2_PICK_AND_PLACE)
- visuals only; collision stays simple boxes, 2 prismatic fingers (no mimic, Gazebo Classic safe)
- finger contact params (kp/kd/minDepth/maxVel)
- PICK_Z 0.085 -> 0.17, PLACE_Z 0.09 -> 0.175 for the new finger geometry
- install meshes via setup.py

Co-Authored-By: Claude Sonnet 5.5 <noreply@anthropic.com>
Claude-Session: https://claude.ai/code/session_01YU8agv91xm8euCzuaef6nj

File: urdf/simple_gripper.xacro (robot description, xacro)
@@ -1,19 +1,31 @@
 <?xml version="1.0"?>
 <robot xmlns:xacro="http://www.ros.org/wiki/xacro">
-  <xacro:property name="finger_length" value="0.06"/>
-  <xacro:property name="finger_width"  value="0.02"/>
-  <xacro:property name="finger_height" value="0.015"/>
-  <xacro:property name="base_size"     value="0.05"/>
+  <!-- Gripper song song 2 ngon truot (khong dung <mimic>, chay duoc tren Gazebo Classic).
+       Hinh dang: adapter + than Robotiq 2F-85 (mesh MIT, xem meshes/robotiq_2f_85/LICENSE.*)
+       Chi dung mesh cho VISUAL; collision la hop don gian de MoveIt/ODE on dinh.
+       Mesh Robotiq mo theo truc x -> xoay 90 do quanh z de ngon mo theo truc y cua tool0. -->
+  <xacro:property name="finger_len"    value="0.06"/>   <!-- doc truc z (dai) -->
+  <xacro:property name="finger_wid"    value="0.02"/>   <!-- doc truc x -->
+  <xacro:property name="finger_thk"    value="0.012"/>  <!-- doc truc y (huong mo) -->
+  <xacro:property name="finger_y0"     value="0.021"/>  <!-- tam ngon khi dong (q=0): mat trong o +-0.015 -->
+  <xacro:property name="finger_z"      value="0.134"/>  <!-- tam ngon duoi tool0; ngon nam duoi than 0.104..0.164 -->
+  <xacro:property name="body_top"      value="0.0139"/> <!-- adapter cao 0.0139 -->
+  <xacro:property name="body_bottom"   value="0.100"/>
   <xacro:property name="max_open"      value="0.04"/>
-  <!-- BASE GRIPPER -->
+  <!-- THAN GRIPPER -->
   <link name="gripper_base_link">
     <visual>
-      <geometry><box size="${base_size} ${base_size} 0.03"/></geometry>
-      <material name="grey"><color rgba="0.3 0.3 0.3 1"/></material>
+      <geometry><mesh filename="package://ur3_llm_control/meshes/robotiq_2f_85/ur_to_robotiq_adapter.dae"/></geometry>
+    </visual>
+    <visual>
+      <origin xyz="0 0 0.011" rpy="0 0 1.5708"/>
+      <geometry><mesh filename="package://ur3_llm_control/meshes/robotiq_2f_85/robotiq_base.dae"/></geometry>
     </visual>
     <collision>
-      <geometry><box size="${base_size} ${base_size} 0.03"/></geometry>
+      <origin xyz="0 0 ${(body_top + body_bottom) / 2}" rpy="0 0 0"/>
+      <geometry><box size="0.075 0.085 ${body_bottom - body_top}"/></geometry>
     </collision>
     <inertial>
+      <origin xyz="0 0 0.05" rpy="0 0 0"/>
       <mass value="0.3"/>
       <inertia ixx="0.0003" iyy="0.0003" izz="0.0003" ixy="0" ixz="0" iyz="0"/>
@@ -23,14 +35,14 @@
     <parent link="tool0"/>
     <child  link="gripper_base_link"/>
-    <origin xyz="0 0 0.015" rpy="0 0 0"/>
+    <origin xyz="0 0 0" rpy="0 0 0"/>
   </joint>
-  <!-- LEFT FINGER -->
+  <!-- NGON TRAI -->
   <link name="left_finger_link">
     <visual>
-      <geometry><box size="${finger_length} ${finger_width} ${finger_height}"/></geometry>
-      <material name="dark_grey"><color rgba="0.15 0.15 0.15 1"/></material>
+      <geometry><box size="${finger_wid} ${finger_thk} ${finger_len}"/></geometry>
+      <material name="finger_dark"><color rgba="0.12 0.12 0.13 1"/></material>
     </visual>
     <collision>
-      <geometry><box size="${finger_length} ${finger_width} ${finger_height}"/></geometry>
+      <geometry><box size="${finger_wid} ${finger_thk} ${finger_len}"/></geometry>
     </collision>
     <inertial>
@@ -42,17 +54,17 @@
     <parent link="gripper_base_link"/>
     <child  link="left_finger_link"/>
-    <origin xyz="0 0.025 0.04" rpy="0 0 0"/>
+    <origin xyz="0 ${finger_y0} ${finger_z}" rpy="0 0 0"/>
     <axis xyz="0 1 0"/>
     <limit lower="0.0" upper="${max_open}" effort="50" velocity="0.05"/>
     <dynamics damping="1.0" friction="0.5"/>
   </joint>
-  <!-- RIGHT FINGER -->
+  <!-- NGON PHAI -->
   <link name="right_finger_link">
     <visual>
-      <geometry><box size="${finger_length} ${finger_width} ${finger_height}"/></geometry>
-      <material name="dark_grey"/>
+      <geometry><box size="${finger_wid} ${finger_thk} ${finger_len}"/></geometry>
+      <material name="finger_dark"/>
     </visual>
     <collision>
-      <geometry><box size="${finger_length} ${finger_width} ${finger_height}"/></geometry>
+      <geometry><box size="${finger_wid} ${finger_thk} ${finger_len}"/></geometry>
     </collision>
     <inertial>
@@ -64,16 +76,20 @@
     <parent link="gripper_base_link"/>
     <child  link="right_finger_link"/>
-    <origin xyz="0 -0.025 0.04" rpy="0 0 0"/>
+    <origin xyz="0 ${-finger_y0} ${finger_z}" rpy="0 0 0"/>
     <axis xyz="0 -1 0"/>
     <limit lower="0.0" upper="${max_open}" effort="50" velocity="0.05"/>
     <dynamics damping="1.0" friction="0.5"/>
   </joint>
-  <!-- GAZEBO CONTACT FRICTION -->
+  <!-- MA SAT / TIEP XUC (tham khao thong so cua darshmenon/UR3_ROS2_PICK_AND_PLACE, MIT) -->
   <gazebo reference="left_finger_link">
     <mu1>50.0</mu1><mu2>50.0</mu2>
+    <kp>1000000.0</kp><kd>100.0</kd>
+    <minDepth>0.001</minDepth><maxVel>0.01</maxVel>
     <material>Gazebo/DarkGrey</material>
   </gazebo>
   <gazebo reference="right_finger_link">
     <mu1>50.0</mu1><mu2>50.0</mu2>
+    <kp>1000000.0</kp><kd>100.0</kd>
+    <minDepth>0.001</minDepth><maxVel>0.01</maxVel>
     <material>Gazebo/DarkGrey</material>
   </gazebo>

Commit message: fix: remove ': ' from xacro comments (breaks rcl YAML parsing of robot_description)
controller_manager failed to start with a parser error because comments in
simple_gripper.xacro contained a colon followed by a space; rcl parses the
robot_description argument as YAML.

Co-Authored-By: Claude Sonnet 5.5 <noreply@anthropic.com>
Claude-Session: https://claude.ai/code/session_01YU8agv91xm8euCzuaef6nj

File: urdf/simple_gripper.xacro (robot description, xacro)
@@ -2,11 +2,13 @@
 <robot xmlns:xacro="http://www.ros.org/wiki/xacro">
   <!-- Gripper song song 2 ngon truot (khong dung <mimic>, chay duoc tren Gazebo Classic).
-       Hinh dang: adapter + than Robotiq 2F-85 (mesh MIT, xem meshes/robotiq_2f_85/LICENSE.*)
-       Chi dung mesh cho VISUAL; collision la hop don gian de MoveIt/ODE on dinh.
+       Hinh dang gripper - adapter + than Robotiq 2F-85 (mesh MIT, xem thu muc meshes/robotiq_2f_85)
+       Chi dung mesh cho VISUAL, collision la hop don gian de MoveIt/ODE on dinh.
+       LUU Y - khong de chuoi hai cham + dau cach trong comment cua file xacro, vi rcl doc
+       robot_description nhu YAML nen se bi loi parser va controller_manager khong khoi dong.
        Mesh Robotiq mo theo truc x -> xoay 90 do quanh z de ngon mo theo truc y cua tool0. -->
   <xacro:property name="finger_len"    value="0.06"/>   <!-- doc truc z (dai) -->
   <xacro:property name="finger_wid"    value="0.02"/>   <!-- doc truc x -->
   <xacro:property name="finger_thk"    value="0.012"/>  <!-- doc truc y (huong mo) -->
-  <xacro:property name="finger_y0"     value="0.021"/>  <!-- tam ngon khi dong (q=0): mat trong o +-0.015 -->
+  <xacro:property name="finger_y0"     value="0.021"/>  <!-- tam ngon khi dong (q=0), mat trong o +-0.015 -->
   <xacro:property name="finger_z"      value="0.134"/>  <!-- tam ngon duoi tool0; ngon nam duoi than 0.104..0.164 -->
   <xacro:property name="body_top"      value="0.0139"/> <!-- adapter cao 0.0139 -->

Commit message: fix: load Robotiq meshes via file://$(find ...) so Gazebo Classic can resolve them
Co-Authored-By: Claude Sonnet 5.5 <noreply@anthropic.com>
Claude-Session: https://claude.ai/code/session_01YU8agv91xm8euCzuaef6nj

File: urdf/simple_gripper.xacro (robot description, xacro)
@@ -18,9 +18,9 @@
   <link name="gripper_base_link">
     <visual>
-      <geometry><mesh filename="package://ur3_llm_control/meshes/robotiq_2f_85/ur_to_robotiq_adapter.dae"/></geometry>
+      <geometry><mesh filename="file://$(find ur3_llm_control)/meshes/robotiq_2f_85/ur_to_robotiq_adapter.dae"/></geometry>
     </visual>
     <visual>
       <origin xyz="0 0 0.011" rpy="0 0 1.5708"/>
-      <geometry><mesh filename="package://ur3_llm_control/meshes/robotiq_2f_85/robotiq_base.dae"/></geometry>
+      <geometry><mesh filename="file://$(find ur3_llm_control)/meshes/robotiq_2f_85/robotiq_base.dae"/></geometry>
     </visual>
     <collision>

Commit message: style: add rail visual between Robotiq body and fingers, thicker fingers
Visual only; finger contact faces stay at +-0.015 so grasp geometry is unchanged.

Co-Authored-By: Claude Sonnet 5.5 <noreply@anthropic.com>
Claude-Session: https://claude.ai/code/session_01YU8agv91xm8euCzuaef6nj

File: urdf/simple_gripper.xacro (robot description, xacro)
@@ -9,6 +9,6 @@
   <xacro:property name="finger_len"    value="0.06"/>   <!-- doc truc z (dai) -->
   <xacro:property name="finger_wid"    value="0.02"/>   <!-- doc truc x -->
-  <xacro:property name="finger_thk"    value="0.012"/>  <!-- doc truc y (huong mo) -->
-  <xacro:property name="finger_y0"     value="0.021"/>  <!-- tam ngon khi dong (q=0), mat trong o +-0.015 -->
+  <xacro:property name="finger_thk"    value="0.016"/>  <!-- doc truc y (huong mo) -->
+  <xacro:property name="finger_y0"     value="0.023"/>  <!-- tam ngon khi dong (q=0), mat trong o +-0.015 -->
   <xacro:property name="finger_z"      value="0.134"/>  <!-- tam ngon duoi tool0; ngon nam duoi than 0.104..0.164 -->
   <xacro:property name="body_top"      value="0.0139"/> <!-- adapter cao 0.0139 -->
@@ -23,4 +23,10 @@
       <origin xyz="0 0 0.011" rpy="0 0 1.5708"/>
       <geometry><mesh filename="file://$(find ur3_llm_control)/meshes/robotiq_2f_85/robotiq_base.dae"/></geometry>
+    </visual>
+    <!-- Thanh ray noi than voi 2 ngon (chi de nhin, khong co collision) -->
+    <visual>
+      <origin xyz="0 0 ${body_bottom + 0.004}" rpy="0 0 0"/>
+      <geometry><box size="0.03 0.15 0.012"/></geometry>
+      <material name="rail_grey"><color rgba="0.22 0.22 0.24 1"/></material>
     </visual>
     <collision>
